File: extras/Orphbot/PCB/Orphbot PCB.kicad_sch (KiCad schematic)
At the start: 0 parts

Commit message: Finished Example PCB
Parts:
- added H1, H2: MountingHole, MountingHole:MountingHole_3.2mm_M3_Pad_Via, symbol Mechanical:MountingHole
- added J1: Barrel_Jack, Connector_BarrelJack:BarrelJack_Horizontal, symbol Connector:Barrel_Jack
- added J2, J3, J4, J5: Screw_Terminal_01x02, WaypointCarePackage:TerminalBlock_KF301-2P_P5.08mm_Blue, symbol Connector:Screw_Terminal_01x02
- added J7: Raspberry_Pi_4, WaypointCarePackage:MODULE_RASPBERRY_PI_ZERO_2_W, symbol Connector:Raspberry_Pi_4
- added J8: Conn_01x10_Pin, Connector_PinHeader_2.54mm:PinHeader_1x10_P2.54mm_Vertical, symbol Connector:Conn_01x10_Pin
- added SW1: KFC7x7_Latching_DPDT, WaypointCarePackage:KFC7x7_Latching_DPDT_Blue, symbol WaypointCarePackage:KFC7x7_Latching_DPDT
- added U1: MPU6050 Module, WaypointCarePackage:LOW_MPU6050_MODULE, symbol WaypointCarePackage:MPU6050_MODULE
- added U10, U11, U6, U7, U8, U9: SK6812 MINI E, WaypointCarePackage:SK6812MINI_E_CORRECTED, symbol WaypointCarePackage:SK6812_MINI_E_CORRECTED
- added U2, U3: DRV8833 MODULE, WaypointCarePackage:DRV8833_MODULE, symbol WaypointCarePackage:DRV8833_MODULE
- added U4: 0.96 OLED 128x64, WaypointCarePackage:128x64OLED, symbol WaypointCarePackage:0.96_OLED_128x64
- added U5: DROK BUCK MODULE, WaypointCarePackage:LOW_DROK_BUCK_MODULE, symbol WaypointCarePackage:DROK_BUCK_MODULE
Connections:
- new net: J3.1 (Pin_1), U2.5 (OUT4)
- new net: J3.2 (Pin_2), U2.4 (OUT3)
- new net: J4.2 (Pin_2), U3.2 (OUT1)
- new net: J4.1 (Pin_1), U3.3 (OUT2)
- new net: J5.2 (Pin_2), U3.4 (OUT3)
- new net: J5.1 (Pin_1), U3.5 (OUT4)
- new net: J2.2 (Pin_2), U2.2 (OUT1)
- new net: J2.1 (Pin_1), U2.3 (OUT2)
- new net: U10.1 (DOUT), U11.3 (DIN)
- new net: U7.1 (DOUT), U8.3 (DIN)
- new net: U6.1 (DOUT), U7.3 (DIN)
- new net: U8.1 (DOUT), U9.3 (DIN)
- new net: U10.3 (DIN), U9.1 (DOUT)
- new net +3.3V: J7.1 (3V3), J7.17 (3V3), J8.2 (Pin_2), U1.1 (VCC), U4.2 (VCC)
- new net +5V: J7.2 (5V), J7.4 (5V), J8.1 (Pin_1), U10.4 (VDD), U11.4 (VDD), U5.5 (OUT+), U6.4 (VDD), U7.4 (VDD), U8.4 (VDD), U9.4 (VDD)
- new net +9V: SW1.3, SW1.6, U2.10 (VCC), U3.10 (VCC), U5.1 (EN), U5.2 (IN+)
- new net +BATT: J1.1, SW1.2, SW1.5
- new net D1_IN1: J7.31 (GPCLK2/GPIO06), U2.12 (IN1)
- new net D1_IN2: J7.33 (GPIO13/PWM1), U2.11 (IN2)
- new net D1_IN3: J7.35 (GPIO19/SPI1_MISO/PCM_FS), U2.8 (IN3)
- new net D1_IN4: J7.37 (GPIO26/SDIO_DAT2), U2.7 (IN4)
- new net D2_IN1: J7.32 (GPIO12/PWM0), U3.12 (IN1)
- new net D2_IN2: J7.36 (GPIO16/SPI1_~{CE2}), U3.11 (IN2)
- new net D2_IN3: J7.38 (GPIO20/SPI1_MOSI/PCM_DIN/PWM1), U3.8 (IN3)
- new net D2_IN4: J7.40 (GPIO21/SPI1_SCLK/PCM_DOUT), U3.7 (IN4)
- new net GND: J1.2, J7.14 (GND), J7.20 (GND), J7.25 (GND), J7.30 (GND), J7.34 (GND), J7.39 (GND), J7.6 (GND), J7.9 (GND), J8.3 (Pin_3), U1.2 (GND), U10.2 (VSS), U11.2 (VSS), U2.9 (GND), U3.9 (GND), U4.1 (GND), U5.3 (In-), U5.4 (OUT-), U6.2 (VSS), U7.2 (VSS), U8.2 (VSS), U9.2 (VSS)
- new net GPIO10: J7.19 (MOSI_SPI0/GPIO10)
- new net GPIO11: J7.23 (SCLK_SPI0/GPIO11)
- new net GPIO14: J7.8 (GPIO14/UART_TXD)
- new net GPIO15: J7.10 (GPIO15/UART_RXD)
- new net GPIO22: J7.15 (GPIO22/SDIO_CLK)
- new net GPIO23: J7.16 (GPIO23/SDIO_CMD)
- new net GPIO24: J7.18 (GPIO24/SDIO_DAT0)
- new net GPIO25: J7.22 (GPIO25/SDIO_DAT1)
- new net GPIO4: J7.7 (GPCLK0/GPIO04), J8.6 (Pin_6)
- new net GPIO5: J7.29 (GPCLK1/GPIO05), J8.7 (Pin_7)
- new net GPIO7: J7.26 (~{CE1}_SPI0/GPIO07), J8.8 (Pin_8)
- new net GPIO8: J7.24 (~{CE0}_SPI0/GPIO08), J8.9 (Pin_9)
- new net GPIO9: J7.21 (MISO_SPI0/GPIO09), J8.10 (Pin_10)
- new net LED_DATA: J7.12 (GPIO18/SPI1_~{CE0}/PCM_CLK/PWM0), U6.3 (DIN)
- new net SCL: J7.5 (SCL_I2C1/GPIO03), J8.5 (Pin_5), U1.3 (SCL), U4.3 (SCL)
- new net SDA: J7.3 (SDA_I2C1/GPIO02), J8.4 (Pin_4), U1.4 (SDA), U4.4 (SDA)
- no-connect marks 0 -> 14
Other:
- note added: "IMU"
- note added: "MOTOR CONTROLLERS"
- note added: "MOUNTING"
- note added: "OLED"
- note added: "PIN HEADER"
- note added: "POWER"
- note added: "RASPBERRY PI"

Commit message: Updated Example PCB
Added servo connector + flipped LEDs to be facing down.
Connections:
- net +5V: now also J8.9 (Pin_9)
- net GND: now also J8.8 (Pin_8)
- net GPIO7: no longer J8.8 (Pin_8)
- net GPIO8: no longer J8.9 (Pin_9)
Changed lines of the file:
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@@
+	)
+	(junction
+		(at 160.02 167.64)
+		(diameter 0)
+		(color 0 0 0 0)
 	)
 	(junction
@@
 	(wire
 		(pts
+			(xy 160.02 180.34) (xy 160.02 167.64)
+		)
+		(stroke
+			(width 0)
+			(type default)
+		)
+	)
+	(wire
+		(pts
 			(xy 195.58 109.22) (xy 195.58 110.49)
 		)
@@
 	(wire
 		(pts
+			(xy 149.86 182.88) (xy 167.64 182.88)
+		)
+		(stroke
+			(width 0)
+			(type default)
+		)
+	)
+	(wire
+		(pts
 			(xy 173.99 109.22) (xy 195.58 109.22)
 		)
@@
 	(wire
 		(pts
+			(xy 149.86 180.34) (xy 160.02 180.34)
+		)
+		(stroke
+			(width 0)
+			(type default)
+		)
+	)
+	(wire
+		(pts
 			(xy 114.3 46.99) (xy 114.3 49.53)
 		)
@@
 	(wire
 		(pts
+			(xy 160.02 167.64) (xy 149.86 167.64)
+		)
+		(stroke
+			(width 0)
+			(type default)
+		)
+	)
+	(wire
+		(pts
 			(xy 106.68 49.53) (xy 107.95 49.53)
 		)
@@
 	(wire
 		(pts
-			(xy 163.83 167.64) (xy 149.86 167.64)
+			(xy 163.83 167.64) (xy 160.02 167.64)
 		)
 		(stroke
@@
 		)
 	)
-	(label "GPIO8"
-		(at 149.86 182.88 0)
-		(effects
-			(font
-				(size 1.27 1.27)
-			)
-			(justify left bottom)
-		)
-	)
 	(label "SCL"
 		(at 31.75 148.59 180)
@@
 			)
 			(justify right bottom)
-		)
-	)
-	(label "GPIO7"
-		(at 149.86 180.34 0)
-		(effects
-			(font
-				(size 1.27 1.27)
-			)
-			(justify left bottom)
 		)
 	)
@@
 					(unit 1)
 				)
+			)
+		)
+	)
+	(symbol
+		(lib_id "power:+5V")
+		(at 167.64 182.88 0)
+		(unit 1)
+		(body_style 1)
+		(exclude_from_sim no)
+		(in_bom yes)
+		(on_board yes)
+		(in_pos_files yes)
+		(dnp no)
+		(fields_autoplaced yes)
+		(property "Reference" "#PWR029"
+			(at 167.64 186.69 0)
+			(hide yes)
+			(show_name no)
+			(do_not_autoplace no)
+			(effects
+				(font
+					(size 1.27 1.27)
+				)
+			)
+		)
+		(property "Value" "+5V"
+			(at 167.64 177.8 0)
+			(show_name no)
+			(do_not_autoplace no)
+			(effects
+				(font
+					(size 1.27 1.27)
+				)
+			)
+		)
+		(property "Footprint" ""
+			(at 167.64 182.88 0)
+			(hide yes)
+			(show_name no)
+			(do_not_autoplace no)
+			(effects
+				(font
+					(size 1.27 1.27)
+				)
+			)
+		)
+		(property "Datasheet" ""
+			(at 167.64 182.88 0)
+			(hide yes)
+			(show_name no)
+			(do_not_autoplace no)
+			(effects
+				(font
+					(size 1.27 1.27)
+				)
+			)
+		)
+		(property "Description" "Power symbol creates a global label with name \"+5V\""
+			(at 167.64 182.88 0)
+			(hide yes)
+			(show_name no)
+			(do_not_autoplace no)
+			(effects
+				(font
+					(size 1.27 1.27)
+				)
+			)
+		)
+		(pin "1"
+		)
+		(instances
+			(project "Orphbot PCB"
+				(path "/131471ea-ff09-449d-948e-8bb493b6ad45"
+					(reference "#PWR029")
+					(unit 1)
+				)

Commit message: Add PCB guide and update example PCB
Large update to the Orphbot PCB and docs.
Connections:
- net GPIO10: no longer names the net of J7.19 (MOSI_SPI0/GPIO10)
- net GPIO11: no longer names the net of J7.23 (SCLK_SPI0/GPIO11)
- net GPIO14: no longer names the net of J7.8 (GPIO14/UART_TXD)
- net GPIO15: no longer names the net of J7.10 (GPIO15/UART_RXD)
- net GPIO22: no longer names the net of J7.15 (GPIO22/SDIO_CLK)
- net GPIO23: no longer names the net of J7.16 (GPIO23/SDIO_CMD)
- net GPIO24: no longer names the net of J7.18 (GPIO24/SDIO_DAT0)
- net GPIO25: no longer names the net of J7.22 (GPIO25/SDIO_DAT1)
- net GPIO7: no longer names the net of J7.26 (~{CE1}_SPI0/GPIO07)
- net GPIO8: no longer names the net of J7.24 (~{CE0}_SPI0/GPIO08)
- no-connect marks 14 -> 24
Other:
- note added: "RGB LEDS"
Changed lines of the file:
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@@
 		)
 	)
-	(text "OLED"
+	(text "RGB LEDS"
 		(exclude_from_sim no)
-		(at 277.114 108.204 0)
+		(at 273.304 108.204 0)
 		(effects
 			(font
@@
 	)
 	(no_connect
+		(at 237.49 77.47)
+	)
+	(no_connect
+		(at 171.45 77.47)
+	)
+	(no_connect
 		(at 53.34 39.37)
 	)
 	(no_connect
+		(at 171.45 46.99)
+	)
+	(no_connect
 		(at 33.02 161.29)
 	)
@@
 	)
 	(no_connect
+		(at 171.45 72.39)
+	)
+	(no_connect
 		(at 171.45 82.55)
 	)
@@
 	)
 	(no_connect
+		(at 171.45 69.85)
+	)
+	(no_connect
+		(at 171.45 44.45)
+	)
+	(no_connect
 		(at 33.02 153.67)
 	)
@@
 	)
 	(no_connect
+		(at 171.45 74.93)
+	)
+	(no_connect
 		(at 33.02 156.21)
 	)
 	(no_connect
+		(at 237.49 80.01)
+	)
+	(no_connect
+		(at 237.49 69.85)
+	)
+	(no_connect
+		(at 237.49 72.39)
+	)
+	(no_connect
 		(at 237.49 44.45)
 	)
@@
 	(wire
 		(pts
-			(xy 170.18 44.45) (xy 171.45 44.45)
-		)
-		(stroke
-			(width 0)
-			(type default)
-		)
-	)
-	(wire
-		(pts
 			(xy 119.38 49.53) (xy 114.3 49.53)
 		)
@@
 	(wire
 		(pts
-			(xy 170.18 72.39) (xy 171.45 72.39)
-		)
-		(stroke
-			(width 0)
-			(type default)
-		)
-	)
-	(wire
-		(pts
-			(xy 238.76 77.47) (xy 237.49 77.47)
-		)
-		(stroke
-			(width 0)
-			(type default)
-		)
-	)
-	(wire
-		(pts
 			(xy 195.58 109.22) (xy 217.17 109.22)
 		)
@@
 	(wire
 		(pts
-			(xy 170.18 46.99) (xy 171.45 46.99)
-		)
-		(stroke
-			(width 0)
-			(type default)
-		)
-	)
-	(wire
-		(pts
 			(xy 203.2 118.11) (xy 209.55 118.11)
 		)
@@
 	(wire
 		(pts
-			(xy 170.18 69.85) (xy 171.45 69.85)
-		)
-		(stroke
-			(width 0)
-			(type default)
-		)
-	)
-	(wire
-		(pts
 			(xy 77.47 101.6) (xy 76.2 101.6)
 		)
@@
 	(wire
 		(pts
-			(xy 170.18 77.47) (xy 171.45 77.47)
-		)
-		(stroke
-			(width 0)
-			(type default)
-		)
-	)
-	(wire
-		(pts
 			(xy 163.83 168.91) (xy 163.83 167.64)
 		)
@@
 	(wire
 		(pts
-			(xy 170.18 74.93) (xy 171.45 74.93)
-		)
-		(stroke
-			(width 0)
-			(type default)
-		)
-	)
-	(wire
-		(pts
-			(xy 238.76 80.01) (xy 237.49 80.01)
-		)
-		(stroke
-			(width 0)
-			(type default)
-		)
-	)
-	(wire
-		(pts
 			(xy 238.76 109.22) (xy 260.35 109.22)
 		)
@@
 	(wire
 		(pts
-			(xy 238.76 69.85) (xy 237.49 69.85)
-		)
-		(stroke
-			(width 0)
-			(type default)
-		)
-	)
-	(wire
-		(pts
 			(xy 35.56 43.18) (xy 39.37 43.18)
 		)
@@
 			(width 0)
 			(type default)
-		)
-	)
-	(wire
-		(pts
-			(xy 238.76 72.39) (xy 237.49 72.39)
-		)
-		(stroke
-			(width 0)
-			(type default)
-		)
-	)
-	(label "GPIO10"
-		(at 238.76 77.47 0)
-		(effects
-			(font
-				(size 1.27 1.27)
-			)
-			(justify left bottom)
 		)
 	)
@@
 		)
 	)
-	(label "GPIO14"
-		(at 170.18 44.45 180)
-		(effects
-			(font
-				(size 1.27 1.27)
-			)
-			(justify right bottom)
-		)
-	)
 	(label "SCL"
 		(at 238.76 54.61 0)
@@
 		)
 	)
-	(label "GPIO7"
-		(at 238.76 69.85 0)
-		(effects
-			(font
-				(size 1.27 1.27)
-			)
-			(justify left bottom)
-		)
-	)
-	(label "GPIO22"
-		(at 170.18 69.85 180)
-		(effects
-			(font
-				(size 1.27 1.27)
-			)
-			(justify right bottom)
-		)
-	)
 	(label "GPIO5"
 		(at 149.86 177.8 0)
@@
 		)
 	)
-	(label "GPIO25"
-		(at 170.18 77.47 180)
-		(effects
-			(font
-				(size 1.27 1.27)
-			)
-			(justify right bottom)
-		)
-	)
 	(label "D2_IN2"
 		(at 77.47 109.22 0)
@@
 		)
 	)
-	(label "GPIO8"
-		(at 238.76 72.39 0)
-		(effects
-			(font
-				(size 1.27 1.27)
-			)
-			(justify left bottom)
-		)
-	)
 	(label "D1_IN2"
 		(at 170.18 39.37 180)
@@
 		)
 	)
-	(label "GPIO11"
-		(at 238.76 80.01 0)
-		(effects
-			(font
-				(size 1.27 1.27)
-			)
-			(justify left bottom)
-		)
-	)
-	(label "GPIO24"
-		(at 170.18 74.93 180)
-		(effects
-			(font
-				(size 1.27 1.27)
-			)
-			(justify right bottom)
-		)
-	)
-	(label "GPIO23"
-		(at 170.18 72.39 180)
-		(effects
-			(font
-				(size 1.27 1.27)
-			)
-			(justify right bottom)
-		)
-	)
 	(label "SDA"
 		(at 31.75 151.13 180)
@@
 		(effects
 			(font
-				(size 1.27 1.27)
-			)
-			(justify right bottom)
-		)
-	)
-	(label "GPIO15"
-		(at 170.18 46.99 180)
-		(effects
-			(font
